File: kicad/ir_beacon/ir_beacon.sch (KiCad schematic (older format))
At the start: 15 parts, among them J1 AVR-ISP-6, Q1 MMBT3904, SW1 On/off, SW2 Timer config, U1 ATtiny85V-10SU

Commit message: Rename files and update README.
Parts:
- J1: symbol roomba_beacon-rescue:AVR-ISP-6-Connector -> ir_beacon-rescue:AVR-ISP-6-Connector
- U1: symbol roomba_beacon-rescue:ATtiny85V-10SU-MCU_Microchip_ATtiny -> ir_beacon-rescue:ATtiny85V-10SU-MCU_Microchip_ATtiny
Other:
- note added: "DIP switch to configure how many \nminutes the device should be active \nbeforing going back to sleep:\n0: always on\n1: 60\n2: 120\n3: 180"
- note removed: "DIP switch to configure how many \nminutes the device should be active \nbeforing going back to sleep:\n0: 60\n1: 120\n2: 180\n4: always on"
Changed lines of the file:
@@
 encoding utf-8
 Sheet 1 1
-Title "Vaccum cleaner IR wall"
+Title "IR beacon for vacuum cleaner"
 Date "2019-11-12"
 Rev "1.0"
@@
 $EndComp
 $Comp
-L roomba_beacon-rescue:ATtiny85V-10SU-MCU_Microchip_ATtiny U1
+L ir_beacon-rescue:ATtiny85V-10SU-MCU_Microchip_ATtiny U1
 U 1 1 5DCA85E8
 P 5200 4900
@@
 IR LED for sending pulses to the \nIR receiver on the vaccum cleaner.
 Text Notes 6800 4350 0    50   ~ 0
-DIP switch to configure how many \nminutes the device should be active \nbeforing going back to sleep:\n0: 60\n1: 120\n2: 180\n4: always on
+DIP switch to configure how many \nminutes the device should be active \nbeforing going back to sleep:\n0: always on\n1: 60\n2: 120\n3: 180
 $Comp
 L power:PWR_FLAG #FLG0101
@@
 ISP (In System Programming) header
 $Comp
-L roomba_beacon-rescue:AVR-ISP-6-Connector J1
+L ir_beacon-rescue:AVR-ISP-6-Connector J1
 U 1 1 5DE603CF
 P 4800 3150
