File: kicad/ir_beacon/ir_beacon.kicad_pcb (KiCad board)
At the start: 2 copper layers, 79.4 x 49.1 mm, 20 parts, among them J1 AVR-ISP-6, Q1 MMBT3904, SW1 On/off, SW2 Timer config, U1 ATtiny85V-10SU

Commit message: Rename files and update README.
Other:
- board text added: "IR beacon v1.0. Per Thomas Jahr 2019"
- board text removed: "Roomba IR stopper v1.0. Per Thomas Jahr 2019"
Changed lines of the file:
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@@
   (gr_line (start 110.503185 72.914734) (end 110.503185 106.737395) (layer Edge.Cuts) (width 0.15))
   (gr_line (start 118.364 65.278) (end 182.005227 65.278) (layer Edge.Cuts) (width 0.15))
-  (gr_text "Roomba IR stopper v1.0.\nPer Thomas Jahr 2019" (at 137.668 110.236) (layer B.SilkS)
+  (gr_text "IR beacon v1.0.\nPer Thomas Jahr 2019" (at 137.668 110.236) (layer B.SilkS)
     (effects (font (size 1 1) (thickness 0.15)) (justify mirror))
   )

Commit message: Cleanup a bit, add images and convert to KiCAD 6.
Parts:
- C1: footprint Capacitor_Tantalum_SMD:CP_EIA-3528-12_Kemet-T_Pad1.50x2.35mm_HandSolder -> Capacitor_Tantalum_SMD:CP_EIA-6032-28_Kemet-C_Pad2.25x2.35mm_HandSolder
Other:
- net class Default removed
